Commit message: Adding swingup and real life

File: rlr_urdf.urdf (robot description, URDF)
Before this commit: robot rlr_urdf, 4 links, 3 joints
Links:
- link base_link: mass 1.1686 -> 1.1848
- link link1: mass 0.27518 -> 0.27755
- link link2: mass 0.064915 -> 0.072015
Joints:
- joint joint1: limit lower=-4.71 upper=4.71 effort=0.07 velocity=46 -> lower=-3.14 upper=3.14 effort=0.07 velocity=46; type revolute -> continuous
